File: mcu.kicad_sch (KiCad schematic)
At the start: 14 parts

Commit message: midsave
Parts:
- removed A?: ESP32, PCM_SL_Development_Boards:DOIT_ESP32_DEVKIT_30Pins, symbol PCM_SL_Development_Board:ESP32_DevKit_V1_DOIT_30GPIOs
- removed C? (x6): 1n, symbol Device:C
- removed C?: 10u, symbol Device:C
- removed R? (x6): 100, symbol Device:R
- added A1: ESP32, PCM_SL_Development_Boards:DOIT_ESP32_DEVKIT_30Pins, symbol PCM_SL_Development_Board:ESP32_DevKit_V1_DOIT_30GPIOs
- added C10, C4, C5, C6, C8, C9: 1n, Capacitor_THT:C_Disc_D4.7mm_W2.5mm_P5.00mm, symbol Device:C
- added C7: 10u, Capacitor_THT:C_Radial_D6.3mm_H5.0mm_P2.50mm, symbol Device:C
- added Q1: BC547, PCM_Package_TO_SOT_THT_AKL:TO-92_HandSolder, symbol PCM_Transistor_BJT_AKL:BC547
- added R1, R2, R3, R4, R5, R6: 100, PCM_Resistor_THT_AKL:R_Axial_DIN0411_L9.9mm_D3.6mm_P20.32mm_Horizontal, symbol Device:R
- added R7: 20k, PCM_Resistor_THT_AKL:R_Axial_DIN0411_L9.9mm_D3.6mm_P20.32mm_Horizontal, symbol Device:R
- added R8: 240, PCM_Resistor_THT_AKL:R_Axial_DIN0411_L9.9mm_D3.6mm_P20.32mm_Horizontal, symbol Device:R
- added U1, U2, U3: 4066, Package_DIP:DIP-14_W7.62mm_LongPads, symbol 4xxx_IEEE:4066
Connections:
- net +5V: now also A1.30 (VIN), C7.1, R8.2, U1.14 (Vdd), U1.14 (Vdd), U1.14 (Vdd), U1.14 (Vdd), U2.14 (Vdd), U2.14 (Vdd), U2.14 (Vdd), U3.14 (Vdd), U3.14 (Vdd), U3.14 (Vdd)
- net GND: now also A1.2 (GND), A1.29 (GND), C10.2, C4.2, C5.2, C6.2, C7.2, C8.2, C9.2, Q1.3 (E), U1.7 (Vss), U1.7 (Vss), U1.7 (Vss), U1.7 (Vss), U2.7 (Vss), U2.7 (Vss), U2.7 (Vss), U3.7 (Vss), U3.7 (Vss), U3.7 (Vss)
- net PWM_UH: now also A1.26 (ADC2_CH6/D14), R3.1
- net PWM_UL: now also A1.23 (DAC1/ADC2_CH8/D25), R6.1
- net PWM_VH: now also A1.27 (ADC2_CH5/D12), R2.1
- net PWM_VL: now also A1.24 (DAC2/ADC2_CH9/D26), R5.1
- net PWM_WH: now also A1.28 (ADC2_CH4/D13), R1.1
- net PWM_WL: now also A1.25 (ADC2_CH7/D27), R4.1
- new net: Q1.2 (B), R7.2
- new net: U2.14 (Vdd), U3.14 (Vdd)
- new net: U2.7 (Vss), U3.7 (Vss)
- new net A_L1_AF/V_L1: A1.22 (ADC1_CH5/D33), U1.10 (O/I), U1.2 (O/I)
- new net A_L1_DF/V_L12: A1.19 (ADC1_CH6/D34), U2.3 (O/I), U3.10 (O/I)
- new net A_L2_AF/V_L2: A1.21 (ADC1_CH4/D32), U1.3 (O/I), U2.10 (O/I)
- new net A_L2_DF/V_L23: A1.18 (ADC1_CH3/VN), U2.9 (O/I), U3.3 (O/I)
- new net A_L3_AF/V_L3: A1.20 (ADC1_CH7/D35), U1.9 (O/I), U2.2 (O/I)
- new net A_L3_DF/V_Link: A1.17 (ADC1_CH0/VP), U3.2 (O/I), U3.9 (O/I)
- new net AmpSens_L1_AF: U1.11 (I/O)
- new net AmpSens_L1_DF: U3.11 (I/O)
- new net AmpSens_L2_AF: U2.11 (I/O)
- new net AmpSens_L2_DF: U3.4 (I/O)
- new net AmpSens_L3_AF: U2.1 (I/O)
- new net AmpSens_L3_DF: U3.8 (I/O)
- new net INUH: C6.1, R3.2
- new net INUL: C10.1, R6.2
- new net INVH: C5.1, R2.2
- new net INVL: C9.1, R5.2
- new net INWH: C4.1, R1.2
- new net INWL: C8.1, R4.2
- new net SELBIT: A1.5 (D4/ADC2_CH0), R7.1, U1.13 (ON), U1.5 (ON), U1.6 (ON), U2.5 (ON), U2.6 (ON), U3.13 (ON)
- new net VFO: A1.9 (D18)
- new net VoltSens_L1: U1.1 (I/O)
- new net VoltSens_L12: U2.4 (I/O)
- new net VoltSens_L2: U1.4 (I/O)
- new net VoltSens_L23: U2.8 (I/O)
- new net VoltSens_L3: U1.8 (I/O)
- new net VoltSens_Link: U3.1 (I/O)
- new net ~{SELBIT}: Q1.1 (C), R8.1, U1.12 (ON), U2.12 (ON), U2.13 (ON), U3.12 (ON), U3.5 (ON), U3.6 (ON)
- no-connect marks 21 -> 11
Other:
- note added: "INVERSOR LÓGICO"
- note added: "MUX ANALÓGICO"
- note added: "SAÍDAS PWM"
- company: (none) -> Autor: José Fonseca
- title: (none) -> Microcontrolador

Commit message: f
Parts:
- removed A1: ESP32, PCM_SL_Development_Boards:DOIT_ESP32_DEVKIT_30Pins, symbol PCM_SL_Development_Board:ESP32_DevKit_V1_DOIT_30GPIOs
- removed Q1: BC547, PCM_Package_TO_SOT_THT_AKL:TO-92_HandSolder, symbol PCM_Transistor_BJT_AKL:BC547
- removed U1, U2, U3: 4066, Package_DIP:DIP-14_W7.62mm_LongPads, symbol 4xxx_IEEE:4066
- added C25, C26, C27, C28, C29, C30, C31: 10u, Capacitor_THT:CP_Radial_D6.3mm_P2.50mm, symbol Device:C_Polarized
- added DZ1: 3v3, Diode_THT:D_DO-15_P15.24mm_Horizontal, symbol PCM_Diode_Zener_AKL:D_Zener_Generic
- added J1, J2, J3, J4, J6, J7: AudioJack2, Connector_Audio:Jack_3.5mm_CUI_SJ1-3525N_Horizontal, symbol Connector_Audio:AudioJack2
- added J10, J11, J12, J13, J9: JST_04, Connector_JST:JST_EH_B4B-EH-A_1x04_P2.50mm_Vertical, symbol PCM_SL_Connectors:JST_04
- added J16: JST_03, Connector_JST:JST_EH_B3B-EH-A_1x03_P2.50mm_Vertical, symbol PCM_SL_Connectors:JST_03
- added R18, R19, R20, R21, R22, R23, R24, R25, R26, R27, R29: 10k, PCM_Resistor_THT_AKL:R_Axial_DIN0411_L9.9mm_D3.6mm_P20.32mm_Horizontal, symbol Device:R
- added R28: 1M, PCM_Resistor_THT_AKL:R_Axial_DIN0411_L9.9mm_D3.6mm_P20.32mm_Horizontal, symbol Device:R
- added U1: ESP32-S3-DevKitC, PCM_Espressif:ESP32-S3-DevKitC, symbol PCM_Espressif:ESP32-S3-DevKitC
- R7: value 20k -> 10k
- R8: value 240 -> 10k
Connections:
- net ~{SELBIT} is gone; now on net +3.3V: R8.1
- net +5V: now also J10.4, J11.4, J12.4, J13.4, J16.2, J9.4, U1.21 (5V); no longer R8.2
- net AmpSens_L1_AF: now also J1.T, U1.41 (GPIO1/ADC1_CH0)
- net AmpSens_L1_DF: now also J4.T, U1.40 (GPIO2/ADC1_CH1)
- net AmpSens_L2_AF: now also J2.T, U1.13 (GPIO3/ADC1_CH2)
- net AmpSens_L2_DF: now also J6.T, U1.4 (GPIO4/ADC1_CH3)
- net AmpSens_L3_AF: now also J3.T, U1.5 (GPIO5/ADC1_CH4)
- net AmpSens_L3_DF: now also J7.T, U1.6 (GPIO6/ADC1_CH5)
- net GND: now also C25.2, C26.2, C27.2, C28.2, C29.2, C30.2, C31.2, DZ1.2 (A), J10.1, J10.2, J11.1, J11.2, J12.1, J12.2, J13.1, J13.2, J16.3, J9.1, J9.2, R19.2, R20.2, R21.2, R25.2, R26.2, R27.2, R29.2, U1.22 (GND), U1.23 (GND), U1.24 (GND), U1.44 (GND)
- net INUH: now also C8.1, R4.2; no longer C6.1, R3.2
- net INVH: now also C4.1, R1.2; no longer C5.1, R2.2
- net INWH: now also C5.1, R2.2; no longer C4.1, R1.2
- net INWL: now also C6.1, R3.2; no longer C8.1, R4.2
- net PWM_UH: now also R4.1, U1.11 (GPIO18/ADC2_CH7); no longer R3.1
- net PWM_UL: now also U1.32 (GPIO35)
- net PWM_VH: now also R1.1, U1.19 (GPIO13/ADC2_CH2); no longer R2.1
- net PWM_VL: now also U1.27 (GPIO21)
- net PWM_WH: now also R2.1, U1.20 (GPIO14/ADC2_CH3); no longer R1.1
- net PWM_WL: now also R3.1, U1.10 (GPIO17/ADC2_CH6); no longer R4.1
- net VFO: now also U1.33 (GPIO36)
- net VoltSens_L1: now also J9.3, U1.7 (GPIO7/ADC1_CH6)
- net VoltSens_L12: now also J12.3, U1.17 (GPIO11/ADC2_CH0)
- net VoltSens_L2: now also J10.3, U1.12 (GPIO8/ADC1_CH7)
- net VoltSens_L23: now also J13.3, U1.18 (GPIO12/ADC2_CH1)
- net VoltSens_L3: now also J11.3, U1.15 (GPIO9/ADC1_CH8)
- net VoltSens_Link: now also C31.1, DZ1.1 (K), R28.2, R29.1, U1.16 (GPIO10/ADC1_CH9)
- net at R7.2: now also C25.1, J1.S, R19.1
- net SELBIT renamed +3.3V
- net +3.3V: now also R18.1, R22.1, R23.1, R24.1, U1.1 (3V3), U1.2 (3V3)
- new net: C27.1, J3.S, R18.2, R21.1
- new net: C29.1, J6.S, R23.2, R26.1
- new net: C30.1, J7.S, R24.2, R27.1
- new net: C26.1, J2.S, R20.1, R8.2
- new net: C28.1, J4.S, R22.2, R25.1
- new net +15V: J16.1
- new net VBUS: R28.1
- no-connect marks 11 -> 12
Other:
- note added: "SENSOR DE TENSAO"
- note added: "SENSORES DE CORRENTE"
- note removed: "INVERSOR LÓGICO"
- note removed: "MUX ANALÓGICO"
- moved on the sheet: C10, C4, C5, C6, C8, C9, R1, R2, R3, R4, R5, R6

Commit message: change conector
Parts:
- J1, J2, J3, J4, J6, J7: footprint Connector_Audio:Jack_3.5mm_CUI_SJ1-3525N_Horizontal -> Connector_Audio:Jack_3.5mm_KoreanHropartsElec_PJ-320D-4A_Horizontal
Changed lines of the file:
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@@
 			)
 		)
-		(property "Footprint" "Connector_Audio:Jack_3.5mm_CUI_SJ1-3525N_Horizontal"
+		(property "Footprint" "Connector_Audio:Jack_3.5mm_KoreanHropartsElec_PJ-320D-4A_Horizontal"
 			(at 149.86 68.58 0)
 			(effects
@@
 			)
 		)
-		(property "Footprint" "Connector_Audio:Jack_3.5mm_CUI_SJ1-3525N_Horizontal"
+		(property "Footprint" "Connector_Audio:Jack_3.5mm_KoreanHropartsElec_PJ-320D-4A_Horizontal"
 			(at 151.13 95.25 0)
 			(effects
@@
 			)
 		)
-		(property "Footprint" "Connector_Audio:Jack_3.5mm_CUI_SJ1-3525N_Horizontal"
+		(property "Footprint" "Connector_Audio:Jack_3.5mm_KoreanHropartsElec_PJ-320D-4A_Horizontal"
 			(at 111.76 69.85 0)
 			(effects
@@
 			)
 		)
-		(property "Footprint" "Connector_Audio:Jack_3.5mm_CUI_SJ1-3525N_Horizontal"
+		(property "Footprint" "Connector_Audio:Jack_3.5mm_KoreanHropartsElec_PJ-320D-4A_Horizontal"
 			(at 111.76 44.45 0)
 			(effects
@@
 			)
 		)
-		(property "Footprint" "Connector_Audio:Jack_3.5mm_CUI_SJ1-3525N_Horizontal"
+		(property "Footprint" "Connector_Audio:Jack_3.5mm_KoreanHropartsElec_PJ-320D-4A_Horizontal"
 			(at 149.86 44.45 0)
 			(effects
@@
 			)
 		)
-		(property "Footprint" "Connector_Audio:Jack_3.5mm_CUI_SJ1-3525N_Horizontal"
+		(property "Footprint" "Connector_Audio:Jack_3.5mm_KoreanHropartsElec_PJ-320D-4A_Horizontal"
 			(at 111.76 95.25 0)
 			(effects

Commit message: lol
Parts:
- R28: value 1M -> 1.2M
Connections:
- no-connect marks 12 -> 18
Other:
- moved on the sheet: C7, J16
Changed lines of the file:
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@@
 	)
 	(no_connect
+		(at 74.93 105.41)
+	)
+	(no_connect
 		(at 24.13 49.53)
 	)
@@
 	)
 	(no_connect
+		(at 74.93 100.33)
+	)
+	(no_connect
 		(at 74.93 39.37)
 	)
@@
 	)
 	(no_connect
+		(at 74.93 113.03)
+	)
+	(no_connect
+		(at 74.93 110.49)
+	)
+	(no_connect
+		(at 74.93 107.95)
+	)
+	(no_connect
+		(at 74.93 102.87)
+	)
+	(no_connect
 		(at 24.13 39.37)
 	)
@@
 	(wire
 		(pts
-			(xy 83.82 120.65) (xy 86.36 120.65)
+			(xy 224.79 120.65) (xy 227.33 120.65)
 		)
 		(stroke
@@
 	(wire
 		(pts
-			(xy 88.9 30.48) (xy 88.9 29.21)
+			(xy 85.09 30.48) (xy 85.09 29.21)
 		)
 		(stroke
@@
 	(wire
 		(pts
-			(xy 80.01 123.19) (xy 86.36 123.19)
+			(xy 220.98 123.19) (xy 227.33 123.19)
 		)
 		(stroke
@@
 	(wire
 		(pts
-			(xy 88.9 38.1) (xy 88.9 39.37)
+			(xy 85.09 38.1) (xy 85.09 39.37)
 		)
 		(stroke
@@
 	(wire
 		(pts
-			(xy 81.28 125.73) (xy 86.36 125.73)
+			(xy 222.25 125.73) (xy 227.33 125.73)
 		)
 		(stroke
@@
 	(text "SENSOR DE TENSAO\n"
 		(exclude_from_sim no)
-		(at 226.06 19.304 0)
+		(at 263.906 20.574 0)
 		(effects
 			(font
@@
 		(dnp no)
 		(property "Reference" "R18"
-			(at 116.586 86.106 0)
+			(at 115.316 86.106 0)
 			(effects
 				(font
@@
 		(dnp no)
 		(property "Reference" "R23"
-			(at 154.686 59.436 0)
+			(at 153.416 59.436 0)
 			(effects
 				(font
@@
 	(symbol
 		(lib_id "power:GND")
-		(at 81.28 125.73 0)
+		(at 222.25 125.73 0)
 		(unit 1)
 		(exclude_from_sim no)
@@
 		(dnp no)
 		(property "Reference" "#PWR061"
-			(at 81.28 132.08 0)
+			(at 222.25 132.08 0)
 			(effects
 				(font
@@
 		)
 		(property "Value" "GND"
-			(at 81.28 129.54 0)
+			(at 222.25 129.54 0)
 			(effects
 				(font
@@
 		)
 		(property "Footprint" ""
-			(at 81.28 125.73 0)
+			(at 222.25 125.73 0)
 			(effects
 				(font
@@
 		)
 		(property "Datasheet" ""
-			(at 81.28 125.73 0)
+			(at 222.25 125.73 0)
 			(effects
 				(font
@@
 		)
 		(property "Description" "Power symbol creates a global label with name \"GND\" , ground"
-			(at 81.28 125.73 0)
+			(at 222.25 125.73 0)
 			(effects
 				(font
@@
 		(dnp no)
 		(property "Reference" "R24"
-			(at 155.956 86.106 0)
+			(at 154.686 86.106 0)
 			(effects
 				(font
@@
 	(symbol
 		(lib_id "power:+15V")
-		(at 83.82 120.65 0)
+		(at 224.79 120.65 0)
 		(unit 1)
 		(exclude_from_sim no)
@@
 		(dnp no)
 		(property "Reference" "#PWR062"
-			(at 83.82 124.46 0)
+			(at 224.79 124.46 0)
 			(effects
 				(font
@@
 		)
 		(property "Value" "+15V"
-			(at 83.566 116.84 0)
+			(at 224.536 116.84 0)
 			(effects
 				(font
@@
 		)
 		(property "Footprint" ""
-			(at 83.82 120.65 0)
+			(at 224.79 120.65 0)
 			(effects
 				(font
@@
 		)
 		(property "Datasheet" ""
-			(at 83.82 120.65 0)
+			(at 224.79 120.65 0)
 			(effects
 				(font
@@
 		)
 		(property "Description" "Power symbol creates a global label with name \"+15V\""
-			(at 83.82 120.65 0)
+			(at 224.79 120.65 0)
 			(effects
 				(font
@@
 	(symbol
 		(lib_id "PCM_SL_Connectors:JST_03")
-		(at 90.17 123.19 0)
+		(at 231.14 123.19 0)
 		(unit 1)
 		(exclude_from_sim no)
@@
 		(dnp no)
 		(property "Reference" "J16"
-			(at 92.456 123.19 0)
+			(at 233.426 123.19 0)
 			(effects
 				(font
@@
 		)
 		(property "Value" "JST_03"
-			(at 92.71 124.4599 0)
+			(at 233.68 124.4599 0)
 			(effects
 				(font
@@
 		)
 		(property "Footprint" "Connector_JST:JST_EH_B3B-EH-A_1x03_P2.50mm_Vertical"
-			(at 90.17 115.57 0)
+			(at 231.14 115.57 0)
 			(effects
 				(font
@@
 		)
 		(property "Datasheet" ""
-			(at 90.17 115.57 0)
+			(at 231.14 115.57 0)
 			(effects
 				(font
@@
 		)
 		(property "Description" "JST Connector  3 pins "
-			(at 90.17 123.19 0)
+			(at 231.14 123.19 0)
 			(effects
 				(font
@@
 	(symbol
 		(lib_id "power:+5V")
-		(at 80.01 123.19 0)
+		(at 220.98 123.19 0)
 		(unit 1)
 		(exclude_from_sim no)
@@
 		(dnp no)
 		(property "Reference" "#PWR060"
-			(at 80.01 127 0)
+			(at 220.98 127 0)
 			(effects
 				(font
@@
 		)
 		(property "Value" "+5V"
-			(at 80.01 119.634 0)
+			(at 220.98 119.634 0)
 			(effects
 				(font
@@
 		)
 		(property "Footprint" ""
-			(at 80.01 123.19 0)
+			(at 220.98 123.19 0)
 			(effects
 				(font
@@
 		)
 		(property "Datasheet" ""
-			(at 80.01 123.19 0)
+			(at 220.98 123.19 0)
 			(effects
 				(font
@@
 		)
 		(property "Description" "Power symbol creates a global label with name \"+5V\""
-			(at 80.01 123.19 0)
+			(at 220.98 123.19 0)
 			(effects
 				(font
@@
 			)
 		)
-		(property "Value" "1M"
+		(property "Value" "1.2M"
 			(at 195.58 31.7499 0)
 			(effects
@@
 	(symbol
 		(lib_id "power:GND")
-		(at 88.9 39.37 0)
+		(at 85.09 39.37 0)
 		(mirror y)
 		(unit 1)
@@
 		(dnp no)
 		(property "Reference" "#PWR027"
-			(at 88.9 45.72 0)
+			(at 85.09 45.72 0)
 			(effects
 				(font
@@
 		)
 		(property "Value" "GND"
-			(at 88.9 43.18 0)
+			(at 85.09 43.18 0)
 			(effects
 				(font
@@
 		)
 		(property "Footprint" ""
-			(at 88.9 39.37 0)
+			(at 85.09 39.37 0)
 			(effects
 				(font
@@
 		)
 		(property "Datasheet" ""
-			(at 88.9 39.37 0)
+			(at 85.09 39.37 0)
 			(effects
 				(font
@@
 		)
 		(property "Description" "Power symbol creates a global label with name \"GND\" , ground"
-			(at 88.9 39.37 0)
+			(at 85.09 39.37 0)
 			(effects
 				(font
@@
 		(dnp no)
 		(property "Reference" "R22"
-			(at 154.686 35.306 0)
+			(at 152.908 35.306 0)
 			(effects
 				(font
@@
 	(symbol
 		(lib_id "Device:C")
-		(at 88.9 34.29 0)
+		(at 85.09 34.29 0)
 		(mirror y)
 		(unit 1)
@@
 		(dnp no)
 		(property "Reference" "C7"
-			(at 85.852 33.274 0)
+			(at 82.042 33.274 0)
 			(effects
 				(font
@@
 		)
 		(property "Value" "10u"
-			(at 85.852 35.814 0)
+			(at 82.042 35.814 0)
 			(effects
 				(font
@@
 		)
 		(property "Footprint" "Capacitor_THT:C_Radial_D6.3mm_H5.0mm_P2.50mm"
-			(at 87.9348 38.1 0)
+			(at 84.1248 38.1 0)
 			(effects
 				(font
@@
 		)
 		(property "Datasheet" "~"
-			(at 88.9 34.29 0)
+			(at 85.09 34.29 0)
 			(effects
 				(font
@@
 		)
 		(property "Description" "Unpolarized capacitor"
-			(at 88.9 34.29 0)
+			(at 85.09 34.29 0)
 			(effects
 				(font
@@
 	(symbol
 		(lib_id "power:+5V")
-		(at 88.9 29.21 0)
+		(at 85.09 29.21 0)
 		(mirror y)
 		(unit 1)
@@
 		(dnp no)
 		(property "Reference" "#PWR026"
-			(at 88.9 33.02 0)
+			(at 85.09 33.02 0)
 			(effects
 				(font
@@
 		)
 		(property "Value" "+5V"
-			(at 88.9 25.654 0)
+			(at 85.09 25.654 0)
 			(effects
 				(font
@@
 		)
 		(property "Footprint" ""
-			(at 88.9 29.21 0)
+			(at 85.09 29.21 0)
 			(effects
 				(font
@@
 		)
 		(property "Datasheet" ""
-			(at 88.9 29.21 0)
+			(at 85.09 29.21 0)
 			(effects
 				(font
@@
 		)
 		(property "Description" "Power symbol creates a global label with name \"+5V\""
-			(at 88.9 29.21 0)
+			(at 85.09 29.21 0)
 			(effects
 				(font
