File: TCC.kicad_pcb (KiCad board)
At the start: 2 copper layers, 222.5 x 163 mm, 90 parts, among them IC1 FSBB30CH60, J10 AudioJack2, J11 JST_04, J12 JST_04, J13 JST_04, J14 JST_04, J15 JST_04, J2 AudioJack2, J3 AudioJack2, J4 AudioJack2, J5 Screw_Terminal_01x02, J6 AudioJack2, J7 AudioJack2, J8 Screw_Terminal_3_P5.00mm, Q1 BC547, U1 4066, U2 4066, U3 4066

Commit message: f
Parts:
- removed A1: ESP32, PCM_SL_Development_Boards:DOIT_ESP32_DEVKIT_30Pins
- removed C20, C21, C22: 1n, Capacitor_THT:C_Disc_D4.7mm_W2.5mm_P5.00mm
- removed D2, D3, D4: ~, Diode_THT:D_DO-15_P15.24mm_Horizontal
- removed Q1: BC547, PCM_Package_TO_SOT_THT_AKL:TO-92_HandSolder
- removed R10, R11, R9: 330, PCM_Resistor_THT_AKL:R_Axial_DIN0411_L9.9mm_D3.6mm_P20.32mm_Horizontal
- removed R14: 47K, PCM_Resistor_THT_AKL:R_Axial_DIN0411_L9.9mm_D3.6mm_P20.32mm_Horizontal
- removed R15, R17: 0.1, PCM_Resistor_THT_AKL:R_Axial_DIN0922_L20.0mm_D9.0mm_P30.48mm_Horizontal
- removed R30: 1M, PCM_Resistor_THT_AKL:R_Axial_DIN0411_L9.9mm_D3.6mm_P20.32mm_Horizontal
- removed R31: 10k, PCM_Resistor_THT_AKL:R_Axial_DIN0411_L9.9mm_D3.6mm_P20.32mm_Horizontal
- removed U2, U3: 4066, Package_DIP:DIP-14_W7.62mm_LongPads
- added H1: MountingHole_M3, MountingHole:MountingHole_3.2mm_M3, F.Cu at (185.6, 127.8)
- added H2: MountingHole_M3, MountingHole:MountingHole_3.2mm_M3, F.Cu at (184.7, 27.3)
- added H3: MountingHole_M3, MountingHole:MountingHole_3.2mm_M3, F.Cu at (25.3, 117.1)
- added H4: MountingHole_M3, MountingHole:MountingHole_3.2mm_M3, F.Cu at (35.3, 26.8)
- added H5: MountingHole_M3, MountingHole:MountingHole_3.2mm_M3, F.Cu at (272.9, 158.2)
- added H6: MountingHole_M3, MountingHole:MountingHole_3.2mm_M3, F.Cu at (211.4, 157.6)
- added H7: MountingHole_M3, MountingHole:MountingHole_3.2mm_M3, F.Cu at (272.6, 26.7)
- added H8: MountingHole_M3, MountingHole:MountingHole_3.2mm_M3, F.Cu at (212.5, 27.2)
- added J1: AudioJack2, Connector_Audio:Jack_3.5mm_CUI_SJ1-3525N_Horizontal, F.Cu at (23.1, 34.2)
- added J16: JST_03, Connector_JST:JST_EH_B3B-EH-A_1x03_P2.50mm_Vertical, F.Cu at (99.6, 127.7)
- added J17: Screw_Terminal_01x02, TerminalBlock_Phoenix:TerminalBlock_Phoenix_MKDS-1,5-2_1x02_P5.00mm_Horizontal, F.Cu at (134.0, 110.5)
- added J9: JST_04, Connector_JST:JST_EH_B4B-EH-A_1x04_P2.50mm_Vertical, F.Cu at (84.1, 127.7)
- J10: value AudioJack2 -> JST_04; footprint Connector_Audio:Jack_3.5mm_CUI_SJ1-3525N_Horizontal -> Connector_JST:JST_EH_B4B-EH-A_1x04_P2.50mm_Vertical
- J14: value JST_04 -> Screw_Terminal_01x02; footprint Connector_JST:JST_EH_B4B-EH-A_1x04_P2.50mm_Vertical -> TerminalBlock_Phoenix:TerminalBlock_Phoenix_MKDS-1,5-2_1x02_P5.00mm_Horizontal
- J15: value JST_04 -> JST_03; footprint Connector_JST:JST_EH_B4B-EH-A_1x04_P2.50mm_Vertical -> Connector_JST:JST_EH_B3B-EH-A_1x03_P2.50mm_Vertical
- R16: value 0.1 -> 11m; footprint PCM_Resistor_THT_AKL:R_Axial_DIN0922_L20.0mm_D9.0mm_P30.48mm_Horizontal -> PCM_Resistor_THT_AKL:R_Bare_Metal_Element_L21.3mm_W4.8mm_P20.30mm
- R28: value 10k -> 1M
- R7: value 20k -> 10k
- R8: value 240 -> 10k
- U1: value 4066 -> ESP32-S3-DevKitC; footprint Package_DIP:DIP-14_W7.62mm_LongPads -> PCM_Espressif:ESP32-S3-DevKitC
- moved R7 171.5 mm to (61.3, 31.7), turned to 180 degrees
- moved U1 171.4 mm to (74.1, 31.9)
- moved J15 150.1 mm to (266.2, 66.7), turned to 90 degrees
- moved C1 150.1 mm to (265.8, 136.2), turned to -90 degrees
- moved C18 147.8 mm to (179.6, 50.7)
- moved J14 141.6 mm to (266.4, 106.1), turned to 90 degrees
- moved R6 134.1 mm to (105.8, 41.2)
- moved R8 128.6 mm to (61.1, 101.7), turned to 180 degrees
- moved C10 127.1 mm to (126.5, 45.2), turned to 180 degrees
- moved R16 123.7 mm to (174.4, 99.6), turned to -90 degrees
- moved R13 123.3 mm to (152.5, 42.7)
- moved R5 121.9 mm to (105.8, 50.2)
- moved C2 117.1 mm to (242.3, 136.2), turned to -90 degrees
- moved C9 116.2 mm to (126.6, 54.2), turned to 180 degrees
- moved R3 106.0 mm to (106.0, 59.2)
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Connections:
- C25 pad 1: GND -> Net-(C25-Pad1)
- C25 pad 2: Net-(C25-Pad2) -> GND
- C26 pad 1: GND -> Net-(C26-Pad1)
- C26 pad 2: Net-(C26-Pad2) -> GND
- C27 pad 1: GND -> Net-(C27-Pad1)
- C27 pad 2: Net-(C27-Pad2) -> GND
- C28 pad 1: GND -> Net-(C28-Pad1)
- C28 pad 2: Net-(C28-Pad2) -> GND
- C29 pad 1: GND -> Net-(C29-Pad1)
- C29 pad 2: Net-(C29-Pad2) -> GND
- C30 pad 1: GND -> Net-(C30-Pad1)
- C30 pad 2: Net-(C30-Pad2) -> GND
- C4 pad 1: INWH -> INVH
- C5 pad 1: INVH -> INWH
- C6 pad 1: INUH -> INWL
- C8 pad 1: INWL -> INUH
- IC1 pad 21: RS1 -> Net-(IC1-NU)
- IC1 pad 22: RS2 -> Net-(IC1-NU)
- IC1 pad 23: RS3 -> Net-(IC1-NU)
- J11 pad 3: VoltSens_L1 -> VoltSens_L3
- J12 pad 3: VoltSens_L2 -> VoltSens_L12
- J13 pad 3: VoltSens_L3 -> VoltSens_L23
- J14 pad 1: GND -> VBUS
- J15 pad 1: GND -> +15V
- J15 pad 2: GND -> +5V
- J15 pad 3: VoltSens_L23 -> GND
- J2 pad S: Net-(C25-Pad2) -> Net-(C26-Pad1)
- J2 pad T: AmpSens_L1_AF -> AmpSens_L2_AF
- J3 pad S: Net-(C26-Pad2) -> Net-(C27-Pad1)
- J3 pad T: AmpSens_L2_AF -> AmpSens_L3_AF
- J4 pad S: Net-(C27-Pad2) -> Net-(C28-Pad1)
- J4 pad T: AmpSens_L3_AF -> AmpSens_L1_DF
- J5 pad 1: AC/N -> AC/L
- J5 pad 2: AC/L -> AC/N
- J6 pad S: Net-(C28-Pad2) -> Net-(C29-Pad1)
- J6 pad T: AmpSens_L1_DF -> AmpSens_L2_DF
- J7 pad S: Net-(C29-Pad2) -> Net-(C30-Pad1)
- J7 pad T: AmpSens_L2_DF -> AmpSens_L3_DF
- J8 pad 1: Net-(IC1-U) -> Net-(IC1-W)
- J8 pad 3: Net-(IC1-W) -> Net-(IC1-U)
- R1 pad 1: PWM_WH -> PWM_VH
- R1 pad 2: INWH -> INVH
- R13 pad 2: Net-(D2-K) -> Net-(IC1-NU)
- R16 pad 1: RS2 -> Net-(IC1-NU)
- R18 pad 2: Net-(C25-Pad2) -> Net-(C27-Pad1)
- R19 pad 1: +3.3V -> Net-(C25-Pad1)
- R19 pad 2: Net-(C26-Pad2) -> GND
- R2 pad 1: PWM_VH -> PWM_WH
- R2 pad 2: INVH -> INWH
- R20 pad 1: +3.3V -> Net-(C26-Pad1)
- R20 pad 2: Net-(C27-Pad2) -> GND
- R21 pad 1: Net-(C25-Pad2) -> Net-(C27-Pad1)
- R22 pad 1: Net-(C26-Pad2) -> +3.3V
- R22 pad 2: GND -> Net-(C28-Pad1)
- R23 pad 1: Net-(C27-Pad2) -> +3.3V
- R23 pad 2: GND -> Net-(C29-Pad1)
- R24 pad 2: Net-(C28-Pad2) -> Net-(C30-Pad1)
- R25 pad 1: +3.3V -> Net-(C28-Pad1)
- R25 pad 2: Net-(C29-Pad2) -> GND
- R26 pad 1: +3.3V -> Net-(C29-Pad1)
- R26 pad 2: Net-(C30-Pad2) -> GND
- R27 pad 1: Net-(C28-Pad2) -> Net-(C30-Pad1)
- R28 pad 1: Net-(C29-Pad2) -> VBUS
- R28 pad 2: GND -> VoltSens_Link
- R29 pad 1: Net-(C30-Pad2) -> VoltSens_Link
- R3 pad 1: PWM_UH -> PWM_WL
- R3 pad 2: INUH -> INWL
- R4 pad 1: PWM_WL -> PWM_UH
- R4 pad 2: INWL -> INUH
- R7 pad 1: SELBIT -> +3.3V
- R7 pad 2: Net-(Q1-B) -> Net-(C25-Pad1)
- R8 pad 1: ~{SELBIT} -> +3.3V
- R8 pad 2: +5V -> Net-(C26-Pad1)
- U1 pad 1: VoltSens_L1 -> +3.3V
- U1 pad 10: A_L1_AF/V_L1 -> PWM_WL
- U1 pad 11: AmpSens_L1_AF -> PWM_UH
- U1 pad 12: ~{SELBIT} -> VoltSens_L2
- U1 pad 13: SELBIT -> AmpSens_L2_AF
- U1 pad 14: +5V -> unconnected-(U1-GPIO46-Pad14)
- U1 pad 2: A_L1_AF/V_L1 -> +3.3V
- U1 pad 3: A_L2_AF/V_L2 -> unconnected-(U1-CHIP_PU-Pad3)
- U1 pad 4: VoltSens_L2 -> AmpSens_L2_DF
- U1 pad 5: SELBIT -> AmpSens_L3_AF
- U1 pad 6: SELBIT -> AmpSens_L3_DF
- U1 pad 7: GND -> VoltSens_L1
- U1 pad 8: VoltSens_L3 -> unconnected-(U1-GPIO15/ADC2_CH4/32K_P-Pad8)
- U1 pad 9: A_L3_AF/V_L3 -> unconnected-(U1-GPIO16/ADC2_CH5/32K_N-Pad9)
Routing:
- net +5V: track 0.00 -> 276.9 mm
- net +15V: track 0.00 -> 217.0 mm
- net AmpSens_L2_DF: track 0.00 -> 144.1 mm
- net AmpSens_L3_AF: track 0.00 -> 132.9 mm
- net AmpSens_L3_DF: track 0.00 -> 117.6 mm
- net +3.3V: track 0.00 -> 114.4 mm
- net VoltSens_L3: track 0.00 -> 100.4 mm, vias 0 -> 2
- net VoltSens_L1: track 0.00 -> 98.4 mm, vias 0 -> 2
- net VoltSens_L23: track 0.00 -> 97.3 mm, vias 0 -> 2
- net AmpSens_L2_AF: track 0.00 -> 96.5 mm
- net VoltSens_L2: track 0.00 -> 96.3 mm, vias 0 -> 2
- net AmpSens_L1_DF: track 0.00 -> 94.5 mm
- net VoltSens_L12: track 0.00 -> 88.8 mm, vias 0 -> 2
- net PWM_WL: track 0.00 -> 85.9 mm
- net INWL: track 0.00 -> 85.1 mm
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- added copper zone on B.Cu, net AC/L
- added copper zone on B.Cu, net AC/N
- added copper zone on B.Cu, net GND
- added copper zone on B.Cu, net VBUS
Other:
- board size 222.5 x 163 mm -> 258.2 x 141.2 mm
- board text added: "INVERSOR DE BANCADA AUTOR: JOSE FONSECA UFPEL | GSIC"

Commit message: vv
Parts:
- moved R13 44.6 mm to (184.4, 73.8), turned to -90 degrees
- moved C23 0.44 mm to (165.2, 59.3)
Routing:
- net Net-(IC1-NU): track 82.1 -> 18.5 mm
- net VFO: track 33.7 -> 71.1 mm, vias 0 -> 2
- net +15V: track 217.0 -> 239.4 mm
- net CSC: track 29.8 -> 28.9 mm

Commit message: change conector
Parts:
- removed C1, C2, C3: 100u/500V, Capacitor_THT:CP_Radial_D22.0mm_P10.00mm_SnapIn
- removed D1: KBPC5010T, Diode_THT:Diode_Bridge_DIGITRON_KBPC_T
- removed H1, H2, H3, H4, H5, H6, H7, H8: MountingHole_M3, MountingHole:MountingHole_3.2mm_M3
- removed J14, J5: Screw_Terminal_01x02, TerminalBlock_Phoenix:TerminalBlock_Phoenix_MKDS-1,5-2_1x02_P5.00mm_Horizontal
- removed J15: JST_03, Connector_JST:JST_EH_B3B-EH-A_1x03_P2.50mm_Vertical
- removed L1, L2: Choke, Inductor_THT:L_CommonMode_Toroid_Vertical_L19.3mm_W10.8mm_Px6.35mm_Py15.24mm_Bourns_8100
- removed PS1: HLK-10M05, Converter_ACDC:Converter_ACDC_Hi-Link_HLK-10Mxx
- removed PS2: HLK-10M15, Converter_ACDC:Converter_ACDC_Hi-Link_HLK-10Mxx
- J1, J2, J3, J4, J6, J7: footprint Connector_Audio:Jack_3.5mm_CUI_SJ1-3525N_Horizontal -> Connector_Audio:Jack_3.5mm_KoreanHropartsElec_PJ-320D-4A_Horizontal
- moved J2 2.91 mm to (26.1, 104.2), turned to 0 degrees
- moved J1 2.87 mm to (26.0, 34.0), turned to 0 degrees
- moved J3 2.86 mm to (26.0, 76.2), turned to 0 degrees
- moved J4 2.86 mm to (26.0, 48.2), turned to 0 degrees
- moved J6 2.86 mm to (26.0, 62.2), turned to 0 degrees
- moved J7 2.86 mm to (26.0, 90.2), turned to 0 degrees
- moved C25 0.86 mm to (36.0, 35.2)
- moved C26 0.86 mm to (36.0, 105.7)
- moved C27 0.86 mm to (36.0, 77.4)
- moved C28 0.86 mm to (36.0, 49.7)
- moved C29 0.86 mm to (36.0, 63.9)
- moved C30 0.86 mm to (36.0, 91.2)
- moved R20 0.52 mm to (41.3, 106.7)
- moved R8 0.52 mm to (61.7, 101.7)
- moved R21 0.36 mm to (41.3, 78.2)
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Routing:
- net AC/L: track 74.4 -> 0.00 mm
- net AC/N: track 66.4 -> 0.00 mm
- net +5V: track 276.9 -> 236.0 mm
- net Net-(PS2--Vout): track 21.6 -> 0.00 mm
- net Net-(PS1--Vout): track 21.2 -> 0.00 mm
- net +15V: track 239.4 -> 219.8 mm
- net Net-(PS2-+Vout): track 14.6 -> 0.00 mm
- net AmpSens_L3_DF: track 117.6 -> 130.8 mm
- net AmpSens_L3_AF: track 132.9 -> 145.6 mm
- net AmpSens_L2_DF: track 144.1 -> 156.2 mm
- net Net-(PS1-+Vout): track 8.83 -> 0.00 mm
- net Net-(C28-Pad1): track 23.2 -> 15.7 mm
- net Net-(C29-Pad1): track 23.4 -> 15.9 mm
- net Net-(C27-Pad1): track 23.2 -> 15.7 mm
- net Net-(C25-Pad1): track 23.2 -> 15.8 mm
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- removed copper zone on B.Cu, net AC/L
- removed copper zone on B.Cu, net AC/N
- removed copper zone on B.Cu, net VBUS
Other:
- board size 258.2 x 141.2 mm -> 171 x 108.6 mm

Commit message: lol
Parts:
- added C1: 100u/500V, Capacitor_THT:CP_Radial_D22.0mm_P10.00mm_SnapIn, F.Cu at (262.6, 133.8)
- added C2: 100u/500V, Capacitor_THT:CP_Radial_D22.0mm_P10.00mm_SnapIn, F.Cu at (239.1, 133.8)
- added C20: 100u/500V, Capacitor_THT:CP_Radial_D22.0mm_P10.00mm_SnapIn, F.Cu at (480.3, 98.0)
- added C21: 100u/500V, Capacitor_THT:CP_Radial_D22.0mm_P10.00mm_SnapIn, F.Cu at (506.3, 98.0)
- added C22: 100u/500V, Capacitor_THT:CP_Radial_D22.0mm_P10.00mm_SnapIn, F.Cu at (532.0, 98.0)
- added C3: 100u/500V, Capacitor_THT:CP_Radial_D22.0mm_P10.00mm_SnapIn, F.Cu at (215.5, 133.8)
- added D1: KBPC5010T, Diode_THT:Diode_Bridge_DIGITRON_KBPC_T, F.Cu at (233.2, 119.6)
- added H1: MountingHole_M3, MountingHole:MountingHole_3.2mm_M3, F.Cu at (471.0, 59.0)
- added H2: MountingHole_M3, MountingHole:MountingHole_3.2mm_M3, F.Cu at (551.0, 59.0)
- added H3: MountingHole_M3, MountingHole:MountingHole_3.2mm_M3, F.Cu at (470.0, 122.0)
- added H4: MountingHole_M3, MountingHole:MountingHole_3.2mm_M3, F.Cu at (552.0, 122.0)
- added H5: MountingHole_M3, MountingHole:MountingHole_3.2mm_M3, F.Cu at (269.7, 155.8)
- added H6: MountingHole_M3, MountingHole:MountingHole_3.2mm_M3, F.Cu at (208.2, 155.2)
- added H7: MountingHole_M3, MountingHole:MountingHole_3.2mm_M3, F.Cu at (269.4, 24.3)
- added H8: MountingHole_M3, MountingHole:MountingHole_3.2mm_M3, F.Cu at (209.3, 24.8)
- added J14: Screw_Terminal_01x02, TerminalBlock_Phoenix:TerminalBlock_Phoenix_MKDS-1,5-2_1x02_P5.00mm_Horizontal, F.Cu at (263.2, 103.7)
- added J15: JST_03, Connector_JST:JST_EH_B3B-EH-A_1x03_P2.50mm_Vertical, F.Cu at (263.0, 64.3)
- added J18: Screw_Terminal_3_P5.00mm, TerminalBlock_Phoenix:TerminalBlock_Phoenix_PT-1,5-3-5.0-H_1x03_P5.00mm_Horizontal, F.Cu at (516.0, 62.0)
- added J19: Screw_Terminal_3_P5.00mm, TerminalBlock_Phoenix:TerminalBlock_Phoenix_PT-1,5-3-5.0-H_1x03_P5.00mm_Horizontal, F.Cu at (531.0, 118.5)
- added J20: Screw_Terminal_3_P5.00mm, TerminalBlock_Phoenix:TerminalBlock_Phoenix_PT-1,5-3-5.0-H_1x03_P5.00mm_Horizontal, F.Cu at (506.0, 118.5)
- added J21: Screw_Terminal_3_P5.00mm, TerminalBlock_Phoenix:TerminalBlock_Phoenix_PT-1,5-3-5.0-H_1x03_P5.00mm_Horizontal, F.Cu at (480.0, 118.5)
- added J5: Screw_Terminal_01x02, TerminalBlock_Phoenix:TerminalBlock_Phoenix_MKDS-1,5-2_1x02_P5.00mm_Horizontal, F.Cu at (218.4, 99.0)
- added L1: Choke, Inductor_THT:L_CommonMode_Toroid_Vertical_L19.3mm_W10.8mm_Px6.35mm_Py15.24mm_Bourns_8100, F.Cu at (259.4, 91.3)
- added L2: Choke, Inductor_THT:L_CommonMode_Toroid_Vertical_L19.3mm_W10.8mm_Px6.35mm_Py15.24mm_Bourns_8100, F.Cu at (259.5, 48.1)
- added L3: 220uH, Inductor_THT:L_Toroid_Vertical_L16.0mm_W8.0mm_P7.62mm, F.Cu at (537.0, 74.2)
- added L4: 220uH, Inductor_THT:L_Toroid_Vertical_L16.0mm_W8.0mm_P7.62mm, F.Cu at (511.0, 74.2)
- added L5: 220uH, Inductor_THT:L_Toroid_Vertical_L16.0mm_W8.0mm_P7.62mm, F.Cu at (485.0, 74.6)
- added PS1: HLK-10M05, Converter_ACDC:Converter_ACDC_Hi-Link_HLK-10Mxx, F.Cu at (208.8, 74.4)
- added PS2: HLK-10M15, Converter_ACDC:Converter_ACDC_Hi-Link_HLK-10Mxx, F.Cu at (208.8, 42.1)
- moved J8 5.95 mm to (151.3, 104.1)
- moved C11 5.95 mm to (158.5, 45.9)
- moved C12 5.95 mm to (149.5, 45.9)
- moved C13 5.95 mm to (140.0, 45.9)
- moved C14 5.95 mm to (170.0, 53.4)
- moved C15 5.95 mm to (157.0, 52.9)
- moved C16 5.95 mm to (148.0, 52.9)
- moved C17 5.95 mm to (139.0, 52.9)
- moved C18 5.95 mm to (181.0, 44.9)
- moved C19 5.95 mm to (181.0, 54.4)
- moved R12 5.95 mm to (135.3, 32.4)
- moved R5 5.95 mm to (107.2, 44.4)
- moved R6 5.95 mm to (107.2, 35.4)
- moved R23 5.95 mm to (63.0, 54.4)
- moved C10 5.95 mm to (127.8, 39.4)
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Routing:
- net (no net): track 0.00 -> 207.0 mm
- net Net-(C20-Pad1): track 0.00 -> 102.1 mm
- net Net-(C21-Pad1): track 0.00 -> 73.4 mm
- net Net-(C22-Pad1): track 0.00 -> 60.9 mm
- net +5V: track 236.0 -> 276.9 mm
- net Net-(J18-Pad3): track 0.00 -> 30.1 mm
- net Net-(J18-Pad1): track 0.00 -> 29.7 mm
- net +15V: track 219.8 -> 239.4 mm
- net Net-(J18-Pad2): track 0.00 -> 12.2 mm
- added copper zone on B.Cu, net (none)
- added copper zone on B.Cu, net VBUS
Other:
- board size 171 x 108.6 mm -> 536 x 141.8 mm

Commit message: final
Parts:
- moved H2 345.8 mm to (207.0, 24.0), turned to 90 degrees
- moved L3 316.9 mm to (222.2, 38.0), turned to 90 degrees
- moved J18 306.0 mm to (210.0, 59.0), turned to -90 degrees
- moved H4 298.9 mm to (270.0, 23.0), turned to 90 degrees
- moved C22 291.2 mm to (246.0, 43.0), turned to 90 degrees
- moved L4 289.0 mm to (222.2, 64.0), turned to 90 degrees
- moved J19 274.8 mm to (266.5, 44.0), turned to 90 degrees
- moved H1 267.8 mm to (207.0, 104.0), turned to 90 degrees
- moved H7 266.3 mm to (25.2, 130.6), turned to 90 degrees
- moved L5 262.9 mm to (222.6, 90.0), turned to 90 degrees
- moved C21 262.0 mm to (246.0, 68.7), turned to 90 degrees
- moved H8 247.5 mm to (25.7, 190.7), turned to 90 degrees
- moved J20 244.6 mm to (266.5, 69.0), turned to 90 degrees
- moved C20 234.4 mm to (246.0, 94.7), turned to 90 degrees
- moved L2 229.9 mm to (49.0, 140.5), turned to 180 degrees
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Other:
- board size 536 x 141.8 mm -> 261.6 x 183.5 mm
